Commit message: Spawned the entity is gazebo

File: src/my_robot_description/urdf/robot.urdf (robot description, URDF)
Before this commit: robot my_robot, 13 links, 12 joints
Links:
- link head: mass None -> 3.0; geometry collision sphere radius=0.18; visual sphere radius=0.025
- link left_arm: mass None -> 2.0; geometry collision cylinder length=0.6 radius=0.1; visual cylinder length=0.6 radius=0.1
- link left_leg: mass None -> 5.0; geometry collision box size=0.2 0.18 0.8; visual box size=0.2 0.18 0.8
- link left_leg_plate: mass None -> 3.0; geometry collision box size=0.6 0.18 0.2; visual box size=0.6 0.18 0.2
- link left_leg_wheel_back: mass None -> 1.5; geometry collision cylinder length=0.05 radius=0.2; visual box size=0.02 0.04 0.05
- link left_leg_wheel_front: mass None -> 1.0; geometry collision cylinder length=0.05 radius=0.17; visual box size=0.02 0.035 0.05
- link right_arm: mass None -> 2.0; geometry collision cylinder length=0.6 radius=0.1; visual cylinder length=0.6 radius=0.1
- link right_leg: mass None -> 5.0; geometry collision box size=0.2 0.18 0.8; visual box size=0.2 0.18 0.8
- link right_leg_plate: mass None -> 3.0; geometry collision box size=0.6 0.18 0.2; visual box size=0.6 0.18 0.2
- link right_leg_wheel_back: mass None -> 1.5; geometry collision cylinder length=0.05 radius=0.2; visual box size=0.02 0.04 0.05
- link right_leg_wheel_front: mass None -> 1.0; geometry collision cylinder length=0.05 radius=0.17; visual box size=0.02 0.035 0.05
- link torso: mass None -> 10.0; geometry collision box size=0.2 0.4 0.8; visual box size=0.2 0.4 0.8

File: src/my_robot_description/urdf/robot.urdf.xacro (robot description, xacro)
@@ -35,4 +35,8 @@
       </geometry>
     </collision>
+    <inertial>
+      <mass value="10.0" />
+      <inertia ixx="0.2667" iyy="0.2333" izz="0.0667" ixy="0.0" iyz="0.0" ixz="0.0" />
+    </inertial>
   </link>
   <!--Head-->
@@ -49,4 +53,8 @@
       </geometry>
     </collision>
+    <inertial>
+      <mass value="3.0" />
+      <inertia ixx="0.0389" iyy="0.0389" izz="0.0389" ixy="0.0" iyz="0.0" ixz="0.0" />
+    </inertial>
     <visual>
       <origin xyz="-0.16 0.06 0.04" />
@@ -77,4 +85,8 @@
       </geometry>
     </collision>
+    <inertial>
+      <mass value="5.0" />
+      <inertia ixx="0.295" iyy="0.283" izz="0.033" ixy="0.0" iyz="0.0" ixz="0.0" />
+    </inertial>
   </link>
   <link name="right_leg">
@@ -90,4 +102,8 @@
       </geometry>
     </collision>
+    <inertial>
+      <mass value="5.0" />
+      <inertia ixx="0.295" iyy="0.283" izz="0.033" ixy="0.0" iyz="0.0" ixz="0.0" />
+    </inertial>
   </link>
   <!--Arms-->
@@ -106,4 +122,9 @@
       </geometry>
     </collision>
+    <inertial>
+      <origin xyz="0 0 -0.3" />
+      <mass value="2.0" />
+      <inertia ixx="0.065" iyy="0.065" izz="0.01" ixy="0.0" iyz="0.0" ixz="0.0" />
+    </inertial>
   </link>
   <link name="right_arm">
@@ -121,4 +142,9 @@
       </geometry>
     </collision>
+    <inertial>
+      <origin xyz="0 0 -0.3" />
+      <mass value="2.0" />
+      <inertia ixx="0.065" iyy="0.065" izz="0.01" ixy="0.0" iyz="0.0" ixz="0.0" />
+    </inertial>
   </link>
   <!--Joints-->
@@ -169,6 +195,11 @@
         </geometry>
       </collision>
+      <inertial>
+        <mass value="3.0" />
+        <inertia ixx="0.022" iyy="0.110" izz="0.095" ixy="0.0" iyz="0.0" ixz="0.0" />
+      </inertial>
     </link>
-    <!--Wheel-->
+    <!--Back
+    wheel-->
     <link name="${prefix}_wheel_back">
       <visual>
@@ -186,4 +217,8 @@
         <material name="steve_wheel" />
       </collision>
+      <inertial>
+        <mass value="1.5" />
+        <inertia ixx="0.0056" iyy="0.0056" izz="0.03" ixy="0.0" iyz="0.0" ixz="0.0" />
+      </inertial>
       <!--Marker-->
       <visual>
@@ -195,4 +230,6 @@
       </visual>
     </link>
+    <!--Front
+    wheel-->
     <link name="${prefix}_wheel_front">
       <visual>
@@ -210,4 +247,8 @@
         <material name="steve_wheel" />
       </collision>
+      <inertial>
+        <mass value="1.0" />
+        <inertia ixx="0.036" iyy="0.036" izz="0.0145" ixy="0.0" iyz="0.0" ixz="0.0" />
+      </inertial>
       <!--Marker-->
       <visual>
@@ -239,5 +280,5 @@
   <xacro:wheel_plate_with_wheels prefix="left_leg" parent="left_leg" side="1" />
   <xacro:wheel_plate_with_wheels prefix="right_leg" parent="right_leg" side="-1" />
-  <joint name="world_to_base" type="fixed">
+  <joint name="world_to_base" type="floating">
     <parent link="world" />
     <child link="torso" />
