Commit message: Finally able to see the robot in rviz

File: src/my_robot_description/urdf/robot.urdf.xacro (robot description, xacro)
@@ -1,21 +1,22 @@
 <?xml version="1.0"?>
 <robot name="my_robot" xmlns:xacro="http://www.ros.org/wiki/xacro">
+  <link name="world" />
   <!-- Base -->
   <link name="base_link">
     <visual>
       <geometry>
-        <box size="0.4 0.3 0.1"/>
+        <box size="0.4 0.3 0.1" />
       </geometry>
     </visual>
     <collision>
       <geometry>
-        <box size="0.4 0.3 0.1"/>
+        <box size="0.4 0.3 0.1" />
       </geometry>
     </collision>
     <inertial>
-      <mass value="5.0"/>
-      <origin xyz="0 0 0"/>
+      <mass value="5.0" />
+      <origin xyz="0 0 0" />
       <inertia ixx="0.1" iyy="0.1" izz="0.1"
-               ixy="0.0" ixz="0.0" iyz="0.0"/>
+        ixy="0.0" ixz="0.0" iyz="0.0" />
     </inertial>
   </link>
@@ -23,11 +24,11 @@
   <link name="left_wheel">
     <visual>
-        <origin rpy="1.5708 0 0"/>
-        <geometry>
-        <cylinder radius="0.1" length="0.02"/>
-        </geometry>
-        <material name="black">
-        <color rgba="0.1 0.1 0.1 1.0"/>
-        </material>
+      <origin rpy="1.5708 0 0" />
+      <geometry>
+        <cylinder radius="0.1" length="0.02" />
+      </geometry>
+      <material name="black">
+        <color rgba="0.1 0.1 0.1 1.0" />
+      </material>
     </visual>
   </link>
@@ -35,31 +36,30 @@
   <link name="right_wheel">
     <visual>
-        <origin rpy="1.5708 0 0"/>
-        <geometry>
-        <cylinder radius="0.1" length="0.02"/>
-        </geometry>
-        <material name="black">
-        <color rgba="0.1 0.1 0.1 1.0"/>
-        </material>
+      <origin rpy="1.5708 0 0" />
+      <geometry>
+        <cylinder radius="0.1" length="0.02" />
+      </geometry>
+      <material name="black">
+        <color rgba="0.1 0.1 0.1 1.0" />
+      </material>
     </visual>
   </link>
   <!-- Joints -->
-<joint name="left_wheel_joint" type="continuous">
-  <parent link="base_link"/>
-  <child link="left_wheel"/>
-  <origin xyz="0 0.175 0"/>
-  <axis xyz="0 1 0"/>
-</joint>
+  <joint name="left_wheel_joint" type="continuous">
+    <parent link="base_link" />
+    <child link="left_wheel" />
+    <origin xyz="0 0.175 0" />
+    <axis xyz="0 1 0" />
+  </joint>
   <joint name="right_wheel_joint" type="continuous">
-    <parent link="base_link"/>
-    <child link="right_wheel"/>
-    <origin xyz="0 -0.175 0"/>
-    <axis xyz="0 1 0"/>
+    <parent link="base_link" />
+    <child link="right_wheel" />
+    <origin xyz="0 -0.175 0" />
+    <axis xyz="0 1 0" />
   </joint>
-<gazebo>
-  <plugin
-    filename="libgz_ros2_control-system.so"
-    name="gz_ros2_control::GazeboSystem">
-  </plugin>
-</gazebo>
+  <joint name="world_to_base" type="fixed">
+    <parent link="world" />
+    <child link="base_link" />
+    <origin xyz="0 0 0" />
+  </joint>
 </robot>

Commit message: Created a custom joint state publisher

File: src/my_robot_description/urdf/robot.urdf.xacro (robot description, xacro)
@@ -2,64 +2,185 @@
 <robot name="my_robot" xmlns:xacro="http://www.ros.org/wiki/xacro">
   <link name="world" />
-  <!-- Base -->
-  <link name="base_link">
+  <material name="steve_skin">
+    <color rgba="0.93 0.80 0.67 1.0" />
+  </material>
+  <material name="steve_shirt">
+    <color rgba="0.40 0.65 0.95 1.0" />
+  </material>
+  <material name="steve_pants">
+    <color rgba="0.20 0.30 0.60 1.0" />
+  </material>
+  <material name="steve_wheel_plate">
+    <color rgba="0.30 0.32 0.35 1.0" />
+  </material>
+  <material name="steve_wheel">
+    <color rgba="0.08 0.08 0.08 1.0" />
+  </material>
+  <material name="white">
+    <color rgba="1 1 1 1" />
+  </material>
+  <material name="red">
+    <color rgba="1 0 0 1" />
+  </material>
+  <link name="torso">
     <visual>
       <geometry>
-        <box size="0.4 0.3 0.1" />
+        <box size="0.2 0.4 0.8" />
       </geometry>
-    </visual>
-    <collision>
-      <geometry>
-        <box size="0.4 0.3 0.1" />
-      </geometry>
-    </collision>
-    <inertial>
-      <mass value="5.0" />
-      <origin xyz="0 0 0" />
-      <inertia ixx="0.1" iyy="0.1" izz="0.1"
-        ixy="0.0" ixz="0.0" iyz="0.0" />
-    </inertial>
-  </link>
-  <!-- Left Wheel -->
-  <link name="left_wheel">
-    <visual>
-      <origin rpy="1.5708 0 0" />
-      <geometry>
-        <cylinder radius="0.1" length="0.02" />
-      </geometry>
-      <material name="black">
-        <color rgba="0.1 0.1 0.1 1.0" />
-      </material>
+      <material name="steve_shirt" />
     </visual>
   </link>
-  <!-- Right Wheel -->
-  <link name="right_wheel">
+  <link name="head">
     <visual>
-      <origin rpy="1.5708 0 0" />
       <geometry>
-        <cylinder radius="0.1" length="0.02" />
+        <sphere radius="0.18" />
       </geometry>
-      <material name="black">
-        <color rgba="0.1 0.1 0.1 1.0" />
-      </material>
+      <material name="steve_skin" />
+    </visual>
+    <visual>
+      <origin xyz="-0.16 0.06 0.04" />
+      <geometry>
+        <sphere radius="0.025" />
+      </geometry>
+      <material name="white" />
+    </visual>
+    <visual>
+      <origin xyz="-0.16 -0.06 0.04" />
+      <geometry>
+        <sphere radius="0.025" />
+      </geometry>
+      <material name="white" />
     </visual>
   </link>
-  <!-- Joints -->
-  <joint name="left_wheel_joint" type="continuous">
-    <parent link="base_link" />
-    <child link="left_wheel" />
-    <origin xyz="0 0.175 0" />
+  <link name="left_leg">
+    <visual>
+      <geometry>
+        <box size="0.2 0.18 0.8" />
+      </geometry>
+      <material name="steve_pants" />
+    </visual>
+  </link>
+  <link name="right_leg">
+    <visual>
+      <geometry>
+        <box size="0.2 0.18 0.8" />
+      </geometry>
+      <material name="steve_pants" />
+    </visual>
+  </link>
+  <link name="left_arm">
+    <visual>
+      <origin xyz="0 0 -0.3" />
+      <geometry>
+        <cylinder radius="0.1" length="0.6" />
+      </geometry>
+      <material name="steve_skin" />
+    </visual>
+  </link>
+  <link name="right_arm">
+    <visual>
+      <origin xyz="0 0 -0.3" />
+      <geometry>
+        <cylinder radius="0.1" length="0.6" />
+      </geometry>
+      <material name="steve_skin" />
+    </visual>
+  </link>
+  <joint name="left_leg_joint" type="fixed">
+    <parent link="torso" />
+    <child link="left_leg" />
+    <origin xyz="0 0.11 -0.8" />
+  </joint>
+  <joint name="right_leg_joint" type="fixed">
+    <parent link="torso" />
+    <child link="right_leg" />
+    <origin xyz="0 -0.11 -0.8" />
+  </joint>
+  <joint name="left_arm_joint" type="revolute">
+    <parent link="torso" />
+    <child link="left_arm" />
+    <origin xyz="0 0.3 0.4" />
     <axis xyz="0 1 0" />
+    <limit lower="-1.57" upper="1.57" effort="10" velocity="2" />
   </joint>
-  <joint name="right_wheel_joint" type="continuous">
-    <parent link="base_link" />
-    <child link="right_wheel" />
-    <origin xyz="0 -0.175 0" />
+  <joint name="right_arm_joint" type="revolute">
+    <parent link="torso" />
+    <child link="right_arm" />
+    <origin xyz="0 -0.3 0.4" />
     <axis xyz="0 1 0" />
+    <limit lower="-1.57" upper="1.57" effort="10" velocity="2" />
   </joint>
+  <joint name="head_and_torso" type="revolute">
+    <parent link="torso" />
+    <child link="head" />
+    <origin xyz="0 0 0.58" />
+    <axis xyz="0 0 1" />
+    <limit lower="-0.785" upper="0.785" effort="2" velocity="0.4" />
+  </joint>
+  <xacro:macro name="wheel_plate_with_wheels" params="prefix parent side">
+    <link name="${prefix}_plate">
+      <visual>
+        <geometry>
+          <box size="0.6 0.18 0.2" />
+        </geometry>
+        <material name="steve_wheel_plate" />
+      </visual>
+    </link>
+    <link name="${prefix}_wheel_back">
+      <visual>
+        <origin rpy="1.5708 0 0" />
+        <geometry>
+          <cylinder radius="0.2" length="0.05" />
+        </geometry>
+        <material name="steve_wheel" />
+      </visual>
+      <visual>
+        <origin xyz="-0.19 ${side*0.05} 0" rpy="1.5708 0 0" />
+        <geometry>
+          <box size="0.02 0.04 0.05" />
+        </geometry>
+        <material name="red" />
+      </visual>
+    </link>
+    <link name="${prefix}_wheel_front">
+      <visual>
+        <origin rpy="1.5708 0 0" />
+        <geometry>
+          <cylinder radius="0.17" length="0.05" />
+        </geometry>
+        <material name="steve_wheel" />
+      </visual>
+      <visual>
+        <origin xyz="-0.16 ${side*0.05} 0" rpy="1.5708 0 0" />
+        <geometry>
+          <box size="0.02 0.035 0.05" />
+        </geometry>
+        <material name="red" />
+      </visual>
+    </link>
+    <joint name="${prefix}_front_wheel_joint" type="continuous">
+      <parent link="${prefix}_plate" />
+      <child link="${prefix}_wheel_front" />
+      <origin xyz="-0.2 ${side * 0.115} -0.03" />
+      <axis xyz="0 1 0" />
+    </joint>
+    <joint name="${prefix}_back_wheel_joint" type="continuous">
+      <parent link="${prefix}_plate" />
+      <child link="${prefix}_wheel_back" />
+      <origin xyz="0.2 ${side * 0.115} 0" />
+      <axis xyz="0 1 0" />
+    </joint>
+    <joint name="${prefix}_plate_joint" type="fixed">
+      <parent link="${parent}" />
+      <child link="${prefix}_plate" />
+      <origin xyz="0 0 -0.5" />
+    </joint>
+  </xacro:macro>
+  <xacro:wheel_plate_with_wheels prefix="left_leg" parent="left_leg" side="1" />
+  <xacro:wheel_plate_with_wheels prefix="right_leg" parent="right_leg" side="-1" />
   <joint name="world_to_base" type="fixed">
     <parent link="world" />
-    <child link="base_link" />
-    <origin xyz="0 0 0" />
+    <child link="torso" />
+    <origin xyz="0 0 1.5" />
   </joint>
 </robot>

Commit message: Implementing collision

File: src/my_robot_description/urdf/robot.urdf.xacro (robot description, xacro)
@@ -30,5 +30,11 @@
       <material name="steve_shirt" />
     </visual>
-  </link>
+    <collision>
+      <geometry>
+        <box size="0.2 0.4 0.8" />
+      </geometry>
+    </collision>
+  </link>
+  <!--Head-->
   <link name="head">
     <visual>
@@ -38,4 +44,9 @@
       <material name="steve_skin" />
     </visual>
+    <collision>
+      <geometry>
+        <sphere radius="0.18" />
+      </geometry>
+    </collision>
     <visual>
       <origin xyz="-0.16 0.06 0.04" />
@@ -53,4 +64,5 @@
     </visual>
   </link>
+  <!--Legs-->
   <link name="left_leg">
     <visual>
@@ -60,4 +72,9 @@
       <material name="steve_pants" />
     </visual>
+    <collision>
+      <geometry>
+        <box size="0.2 0.18 0.8" />
+      </geometry>
+    </collision>
   </link>
   <link name="right_leg">
@@ -68,5 +85,11 @@
       <material name="steve_pants" />
     </visual>
-  </link>
+    <collision>
+      <geometry>
+        <box size="0.2 0.18 0.8" />
+      </geometry>
+    </collision>
+  </link>
+  <!--Arms-->
   <link name="left_arm">
     <visual>
@@ -77,4 +100,10 @@
       <material name="steve_skin" />
     </visual>
+    <collision>
+      <origin xyz="0 0 -0.3" />
+      <geometry>
+        <cylinder radius="0.1" length="0.6" />
+      </geometry>
+    </collision>
   </link>
   <link name="right_arm">
@@ -86,5 +115,12 @@
       <material name="steve_skin" />
     </visual>
-  </link>
+    <collision>
+      <origin xyz="0 0 -0.3" />
+      <geometry>
+        <cylinder radius="0.1" length="0.6" />
+      </geometry>
+    </collision>
+  </link>
+  <!--Joints-->
   <joint name="left_leg_joint" type="fixed">
     <parent link="torso" />
@@ -118,4 +154,6 @@
     <limit lower="-0.785" upper="0.785" effort="2" velocity="0.4" />
   </joint>
+  <!--Learning
+  to use xacro macros -->
   <xacro:macro name="wheel_plate_with_wheels" params="prefix parent side">
     <link name="${prefix}_plate">
@@ -126,5 +164,11 @@
         <material name="steve_wheel_plate" />
       </visual>
+      <collision>
+        <geometry>
+          <box size="0.6 0.18 0.2" />
+        </geometry>
+      </collision>
     </link>
+    <!--Wheel-->
     <link name="${prefix}_wheel_back">
       <visual>
@@ -135,4 +179,12 @@
         <material name="steve_wheel" />
       </visual>
+      <collision>
+        <origin rpy="1.5708 0 0" />
+        <geometry>
+          <cylinder radius="0.2" length="0.05" />
+        </geometry>
+        <material name="steve_wheel" />
+      </collision>
+      <!--Marker-->
       <visual>
         <origin xyz="-0.19 ${side*0.05} 0" rpy="1.5708 0 0" />
@@ -151,4 +203,12 @@
         <material name="steve_wheel" />
       </visual>
+      <collision>
+        <origin rpy="1.5708 0 0" />
+        <geometry>
+          <cylinder radius="0.17" length="0.05" />
+        </geometry>
+        <material name="steve_wheel" />
+      </collision>
+      <!--Marker-->
       <visual>
         <origin xyz="-0.16 ${side*0.05} 0" rpy="1.5708 0 0" />

Commit message: 1st commit

File: src/my_robot_description/urdf/robot.urdf.xacro (robot description, xacro)
@@ -5,10 +5,10 @@
     <visual>
       <geometry>
-        <box size="0.4 0.3 0.1"/>
+        <box size="0.6 0.3 0.1"/>
       </geometry>
     </visual>
     <collision>
       <geometry>
-        <box size="0.4 0.3 0.1"/>
+        <box size="0.6 0.3 0.1"/>
       </geometry>
     </collision>
@@ -20,6 +20,20 @@
     </inertial>
   </link>
-  <!-- Left Wheel -->
-  <link name="left_wheel">
+  <!-- Left Behind Wheel -->
+  <link name="left_behind_wheel">
+    <visual>
+        <origin rpy="1.5708 0 0"/>
+        <geometry>
+        <cylinder radius="0.1" length="0.02"/>
+        </geometry>
+        <material name="black">
+        <color rgba="0.1 0.1 0.1 1.0"/>
+        </material>
+    </visual>
+    <inertial>
+      <mass value = "0.1"/>
+  </link>
+  <!-- Right Behind Wheel -->
+  <link name="right_behind_wheel">
     <visual>
         <origin rpy="1.5708 0 0"/>
@@ -32,6 +46,18 @@
     </visual>
   </link>
-  <!-- Right Wheel -->
-  <link name="right_wheel">
+  <!-- Left Front Wheel -->
+  <link name="left_front_wheel">
+    <visual>
+        <origin rpy="1.5708 0 0"/>
+        <geometry>
+        <cylinder radius="0.1" length="0.02"/>
+        </geometry>
+        <material name="black">
+        <color rgba="0.1 0.1 0.1 1.0"/>
+        </material>
+    </visual>
+  </link>
+  <!-- Right Front Wheel -->
+  <link name="right_front_wheel">
     <visual>
         <origin rpy="1.5708 0 0"/>
@@ -45,14 +71,26 @@
   </link>
   <!-- Joints -->
-<joint name="left_wheel_joint" type="continuous">
-  <parent link="base_link"/>
-  <child link="left_wheel"/>
-  <origin xyz="0 0.175 0"/>
-  <axis xyz="0 1 0"/>
-</joint>
-  <joint name="right_wheel_joint" type="continuous">
+  <joint name="left_behind_wheel_joint" type="continuous">
     <parent link="base_link"/>
-    <child link="right_wheel"/>
-    <origin xyz="0 -0.175 0"/>
+    <child link="left_behind_wheel"/>
+    <origin xyz="-0.2 0.175 0"/>
+    <axis xyz="0 1 0"/>
+  </joint>
+  <joint name="right_behind_wheel_joint" type="continuous">
+    <parent link="base_link"/>
+    <child link="right_behind_wheel"/>
+    <origin xyz="-0.2 -0.175 0"/>
+    <axis xyz="0 1 0"/>
+  </joint>
+  <joint name="left_front_wheel_joint" type="continuous">
+    <parent link="base_link"/>
+    <child link="left_front_wheel"/>
+    <origin xyz="0.2 0.175 0"/>
+    <axis xyz="0 1 0"/>
+  </joint>
+  <joint name="right_front_wheel_joint" type="continuous">
+    <parent link="base_link"/>
+    <child link="right_front_wheel"/>
+    <origin xyz="0.2 -0.175 0"/>
     <axis xyz="0 1 0"/>
   </joint>

Commit message: WIP

File: src/my_robot_description/urdf/robot.urdf.xacro (robot description, xacro)
@@ -1,5 +1,6 @@
 <?xml version="1.0"?>
 <robot name="my_robot" xmlns:xacro="http://www.ros.org/wiki/xacro">
-  <link name="world" />
+  <!--<link
+  name="world" />-->
   <material name="steve_skin">
     <color rgba="0.93 0.80 0.67 1.0" />
@@ -280,4 +281,5 @@
   <xacro:wheel_plate_with_wheels prefix="left_leg" parent="left_leg" side="1" />
   <xacro:wheel_plate_with_wheels prefix="right_leg" parent="right_leg" side="-1" />
+  <!--
   <joint name="world_to_base" type="floating">
     <parent link="world" />
@@ -285,3 +287,4 @@
     <origin xyz="0 0 1.5" />
   </joint>
+-->
 </robot>
